Commit message: Switch to ROS2 Humble and integrate ros2_control

File: ROS2/bpl_alpha_description/urdf/alpha_5.urdf.xacro (robot description, xacro)
@@ -13,4 +13,9 @@
         <link name="${name}_base_link"/>
         <link name="${name}_m3_inline_link">
+            <inertial>
+                <origin xyz="2 0 0" />
+                <mass value="1.0" />
+                <inertia  ixx="0.001" ixy="0.0"  ixz="0.0"  iyy="0.001"  iyz="0.0"  izz="0.0001" />
+            </inertial>
             <visual>
                 <geometry>
@@ -22,7 +27,9 @@
             <collision>
                 <geometry>
-                    <cylinder length="0.150" radius="0.020" />
-                </geometry>
-                <origin rpy="0 1.57075 0" xyz="-0.075 0 0" />
+                    <!-- <cylinder length="0.150" radius="0.020" /> -->
+                    <mesh filename="package://bpl_alpha_description/meshes/M3-INLINE.stl"/>
+                </geometry>
+                <!-- <origin rpy="0 1.57075 0" xyz="-0.075 0 0" /> -->
+                <origin rpy="0 0 0" xyz="0 0 0"/>
             </collision>
         </link>
@@ -33,14 +40,22 @@
         </joint>
         <link name="${name}_m2_1_1_link">
+            <inertial>
+                <origin xyz="2 0 0" />
+                <mass value="1.0" />
+                <inertia  ixx="0.001" ixy="0.0"  ixz="0.0"  iyy="0.001"  iyz="0.0"  izz="0.0001" />
+            </inertial>
             <visual>
                 <geometry>
                     <mesh filename="package://bpl_alpha_description/meshes/M2-1-1.stl"/>
-                </geometry>
-                <origin rpy="0 0 0" xyz="0 0 0"/>
-                <material name="${name}_black"/>
-            </visual>
-            <collision>
-                <geometry>
-                    <cylinder length="0.066" radius="0.020" />
+                    <!-- <mesh filename="/workspaces/reach_robotics_sdk_humble/ROS2/bpl_alpha_description/meshes/M2-1-1.stl"/> -->
+                </geometry>
+                <origin rpy="0 0 0" xyz="0 0 0"/>
+                <material name="${name}_black"/>
+            </visual>
+            <collision>
+                <geometry>
+                    <!-- <cylinder length="0.066" radius="0.020" /> -->
+                    <mesh filename="package://bpl_alpha_description/meshes/M2-1-1.stl"/>
+                    <!-- <mesh filename="/workspaces/reach_robotics_sdk_humble/ROS2/bpl_alpha_description/meshes/M2-1-1.stl"/> -->
                 </geometry>
                 <origin rpy="0 0 0" xyz="0 0 0.000" />
@@ -53,6 +68,12 @@
             <axis xyz="0 0 1"/>
             <limit effort="9.0" lower="0.0" upper="6.3" velocity="0.5"/>
+            <dynamics damping="10.0" friction="10.0"/>
         </joint>
         <link name="${name}_m2_joint_link">
+            <inertial>
+                <origin xyz="2 0 0" />
+                <mass value="1.0" />
+                <inertia  ixx="0.001" ixy="0.0"  ixz="0.0"  iyy="0.001"  iyz="0.0"  izz="0.0001" />
+            </inertial>
             <visual>
                 <geometry>
@@ -64,9 +85,11 @@
             <collision>
                 <geometry>
-                    <cylinder length="0.145" radius="0.020" />
-                </geometry>
-                <origin rpy="0 0 0" xyz="-0.02 0 -0.0725" />
-            </collision>
-            <collision>
+                    <!-- <cylinder length="0.145" radius="0.020" /> -->
+                    <mesh filename="package://bpl_alpha_description/meshes/M2.stl"/>
+                </geometry>
+                <!-- <origin rpy="0 0 0" xyz="-0.02 0 -0.0725" /> -->
+                <origin rpy="0 0 0" xyz="0 0 0"/>
+            </collision>
+            <!-- <collision>
                 <geometry>
                     <cylinder length="0.040" radius="0.020" />
@@ -79,5 +102,5 @@
                 </geometry>
                 <origin rpy="1.5707 0 0" xyz="-0.040 0 -0.1453" />
-            </collision>
+            </collision> -->
         </link>
         <joint name="${name}_axis_d" type="revolute">
@@ -86,7 +109,13 @@
             <origin xyz="-0.02 0 0.033"/>
             <axis xyz="0 1 0"/>
-            <limit effort="9.0" lower="0.0" upper="3.8" velocity="0.5"/>
+            <limit effort="9.0" lower="0" upper="3.8" velocity="0.5"/>
+            <dynamics damping="10.0" friction="10.0"/>
         </joint>
         <link name="${name}_m2_1_2_link">
+            <inertial>
+                <origin xyz="2 0 0" />
+                <mass value="1.0" />
+                <inertia  ixx="0.001" ixy="0.0"  ixz="0.0"  iyy="0.001"  iyz="0.0"  izz="0.0001" />
+            </inertial>
             <visual>
                 <geometry>
@@ -98,7 +127,9 @@
             <collision>
                 <geometry>
-                    <cylinder length="0.033" radius="0.020" />
-                </geometry>
-                <origin rpy="0 0 0" xyz="0.02 0 0.0165" />
+                    <!-- <cylinder length="0.033" radius="0.020" /> -->
+                    <mesh filename="package://bpl_alpha_description/meshes/M2-1-3.stl"/>
+                </geometry>
+                <!-- <origin rpy="0 0 0" xyz="0.02 0 0.0165" /> -->
+                <origin rpy="0 0 0" xyz="0 0 0"/>
             </collision>
         </link>
@@ -109,6 +140,12 @@
             <axis xyz="0 1 0"/>
             <limit effort="9.0" lower="0.0" upper="3.5" velocity="0.5"/>
+            <dynamics damping="10.0" friction="10.0"/>
         </joint>
         <link name="${name}_m1_link">
+            <inertial>
+                <origin xyz="2 0 0" />
+                <mass value="1.0" />
+                <inertia  ixx="0.001" ixy="0.0"  ixz="0.0"  iyy="0.001"  iyz="0.0"  izz="0.0001" />
+            </inertial>
             <visual>
                 <geometry>
@@ -120,10 +157,12 @@
             <collision>
                 <geometry>
-                    <cylinder length="0.10975" radius="0.020" />
-                </geometry>
-                <origin rpy="0 0 0" xyz="0.00 0 0.054875" />
-            </collision>
-        </link>
-            <joint name="${name}_axis_b" type="revolute">
+                    <!-- <cylinder length="0.10975" radius="0.020" /> -->
+                    <mesh filename="package://bpl_alpha_description/meshes/RS1-100-101-123.stl"/>
+                </geometry>
+                <!-- <origin rpy="0 0 0" xyz="0.00 0 0.054875" /> -->
+                <origin rpy="0 -1.5707 0" xyz="0 0 0"/>
+            </collision>
+        </link>
+        <joint name="${name}_axis_b" type="revolute">
             <parent link="${name}_m2_1_2_link"/>
             <child link="${name}_m1_link"/>
@@ -131,4 +170,5 @@
             <axis xyz="0 0 -1"/>
             <limit effort="9.0" lower="0.0" upper="6.2" velocity="0.5"/>
+            <dynamics damping="10.0" friction="10.0"/>
         </joint>
         <material name="${name}_jaws_black">
@@ -141,6 +181,17 @@
         </joint>
         <link name="${name}_jaws_base_link">
-        </link>
-        <link name="${name}_push_rod"/>
+            <inertial>
+                <origin xyz="2 0 0" />
+                <mass value="1.0" />
+                <inertia  ixx="0.001" ixy="0.0"  ixz="0.0"  iyy="0.001"  iyz="0.0"  izz="0.0001" />
+            </inertial>
+        </link>
+        <link name="${name}_push_rod">
+            <inertial>
+                <origin xyz="2 0 0" />
+                <mass value="1.0" />
+                <inertia  ixx="0.001" ixy="0.0"  ixz="0.0"  iyy="0.001"  iyz="0.0"  izz="0.0001" />
+            </inertial>
+        </link>
         <joint name="${name}_axis_a" type="prismatic">
             <origin rpy="0 0 0" xyz="0 0 0.009"/>
@@ -149,4 +200,5 @@
             <axis xyz="0 0 1"/>
             <limit effort="10" lower="0" upper="0.015" velocity="10"/>
+            <dynamics damping="10.0" friction="10.0"/>
         </joint>
         <xacro:include filename="$(find bpl_alpha_description)/urdf/end_effectors/standard_jaws.urdf.xacro"/>
@@ -154,4 +206,6 @@
             <origin xyz="0 0 0" rpy="0 0 0"/>
         </xacro:alpha_standard_jaws>
+        <xacro:include filename='alpha_5_gazebo.xacro'/>
+        <xacro:include filename='ros2_control.xacro'/>
     </xacro:macro>
 </robot>

File: ROS2/bpl_alpha_description/urdf/alpha_5_example.urdf.xacro (robot description, xacro)
@@ -3,6 +3,13 @@
   <xacro:include filename="$(find bpl_alpha_description)/urdf/alpha_5.urdf.xacro"/>
     <link name="base_link"/>
+    <link name="world"/>
+    <joint name="fixed_to_world" type="fixed">
+      <parent link="world"/>
+      <child link="base_link"/>
+      <origin xyz="0 0 0" rpy="0 0 0"/>
+    </joint>
     <xacro:alpha_5 parent="base_link" name="alpha">
       <origin xyz="0 0 0" rpy="0 0 0"/>
     </xacro:alpha_5>
+  <xacro:include filename="ros2_control.xacro" />
 </robot>

File: ROS2/bpl_alpha_description/urdf/end_effectors/standard_jaws.urdf.xacro (robot description, xacro)
@@ -18,4 +18,9 @@
                 <material name="${name}_black"/>
             </visual>
+            <inertial>
+                <origin xyz="2 0 0" />
+                <mass value="1.0" />
+                <inertia  ixx="0.001" ixy="0.0"  ixz="0.0"  iyy="0.001"  iyz="0.0"  izz="0.0001" />
+            </inertial>
         </link>
         <link name="${name}_rs1_130_link">
@@ -29,8 +34,14 @@
             <collision>
                 <geometry>
-                    <box size="0.012 0.03 0.09"/>
+                    <mesh filename="package://bpl_alpha_description/meshes/end_effectors/RS1-130.stl"/>
+                    <!-- <box size="0.012 0.03 0.09"/> -->
                 </geometry>
                 <origin xyz="0.0 -0.008 0.045" rpy="0 0 0"/>
             </collision>
+            <inertial>
+                <origin xyz="2 0 0" />
+                <mass value="1.0" />
+                <inertia  ixx="0.001" ixy="0.0"  ixz="0.0"  iyy="0.001"  iyz="0.0"  izz="0.0001" />
+            </inertial>
         </link>
         <joint name="${name}_rs1_130_joint" type="revolute">
@@ -52,8 +63,14 @@
             <collision>
                 <geometry>
-                    <box size="0.012 0.03 0.09"/>
+                    <mesh filename="package://bpl_alpha_description/meshes/end_effectors/RS1-139.stl"/>
+                    <!-- <box size="0.012 0.03 0.09"/> -->
                 </geometry>
                 <origin xyz="0.0 0.008 0.045" rpy="0 0 0"/>
             </collision>
+            <inertial>
+                <origin xyz="2 0 0" />
+                <mass value="1.0" />
+                <inertia  ixx="0.001" ixy="0.0"  ixz="0.0"  iyy="0.001"  iyz="0.0"  izz="0.0001" />
+            </inertial>
         </link>
         <joint name="${name}_rs1_139_joint" type="revolute">
