Commit message: Add ros2_control integration files to bpl_alpha_description package

File: ROS2/bpl_alpha_description/urdf/alpha_5.urdf.xacro (robot description, xacro)
@@ -1,157 +1,322 @@
 <?xml version="1.0"?>
 <robot name="alpha_5" xmlns:xacro="http://ros.org/wiki/xacro">
-    <xacro:macro name="alpha_5" params="parent *origin name:=alpha_5">
-        <joint name="${name}_joint" type="fixed">
-            <xacro:insert_block name="origin" />
-            <parent link="${parent}"/>
-            <child link="${name}_base_link" />
+    <material name="black">
+        <color rgba="0.5 0.5 0.5 1.0"/>
+    </material>
+    <link name="world"/>
+    <joint name="world_to_base" type="fixed">
+        <parent link="world"/>
+        <child link="base_link"/>
+        <origin xyz="0 0 0" rpy="0 0 0"/>
+    </joint>
+    <link name="base_link">
+        <inertial>
+            <mass value="1.0" />
+              <inertia ixx="0.001" iyy="0.001" izz="0.001"
+                       ixy="0.0" ixz="0.0" iyz="0.0" />
+        </inertial>
+    </link>
+    <link name="m3_inline_link">
+        <inertial>
+            <mass value="0.5" />
+            <inertia  ixx="0.001" ixy="0.0"  ixz="0.0"
+                      iyy="0.001"  iyz="0.0"  izz="0.0001" />
+        </inertial>
+        <visual>
+            <geometry>
+                <mesh filename="package://bpl_alpha_description/meshes/M3-INLINE.stl"/>
+            </geometry>
+            <origin rpy="0 0 0" xyz="0 0 0"/>
+            <material name="black"/>
+        </visual>
+        <collision>
+            <geometry>
+                <cylinder length="0.150" radius="0.020" />
+            </geometry>
+            <origin rpy="0 1.57075 0" xyz="-0.075 0 0" />
+        </collision>
+    </link>
+    <joint name="base_link_joint" type="fixed">
+        <parent link="base_link"/>
+        <child link="m3_inline_link"/>
+        <origin rpy="0 0 0"/>
+    </joint>
+    <link name="m2_1_1_link">
+        <inertial>
+            <mass value="0.5" />
+            <inertia  ixx="0.001" ixy="0.0"  ixz="0.0"  iyy="0.001"  iyz="0.0"  izz="0.0001" />
+        </inertial>
+        <visual>
+            <geometry>
+                <mesh filename="package://bpl_alpha_description/meshes/M2-1-1.stl"/>
+            </geometry>
+            <origin rpy="0 0 0" xyz="0 0 0.000" />
+            <material name="black"/>
+        </visual>
+        <collision>
+            <geometry>
+                <cylinder length="0.066" radius="0.020" />
+            </geometry>
+            <origin rpy="0 0 0" xyz="0 0 0.000" />
+        </collision>
+    </link>
+    <joint name="axis_e" type="revolute">
+        <parent link="m3_inline_link"/>
+        <child link="m2_1_1_link"/>
+        <origin xyz="0 0 0.014"/>
+        <axis xyz="0 0 1"/>
+        <limit effort="25" lower="0.0" upper="6.3" velocity="4.0"/>
+        <dynamics damping="0.1"/>
+    </joint>
+    <link name="m2_joint_link">
+        <inertial>
+            <mass value="0.5" />
+            <inertia  ixx="0.001" ixy="0.0"  ixz="0.0"  iyy="0.001"  iyz="0.0"  izz="0.0001" />
+        </inertial>
+        <visual>
+            <geometry>
+                <mesh filename="package://bpl_alpha_description/meshes/M2.stl"/>
+            </geometry>
+            <origin rpy="0 0 0" xyz="0 0 0"/>
+            <material name="black"/>
+        </visual>
+        <collision>
+            <geometry>
+                <cylinder length="0.145" radius="0.020" />
+            </geometry>
+            <origin rpy="0 0 0" xyz="-0.02 0 -0.0725" />
+        </collision>
+        <collision>
+            <geometry>
+                <cylinder length="0.040" radius="0.020" />
+            </geometry>
+            <origin rpy="1.5707 0 0" xyz="0 0 0" />
+        </collision>
+        <collision>
+            <geometry>
+                <cylinder length="0.040" radius="0.020" />
+            </geometry>
+            <origin rpy="1.5707 0 0" xyz="-0.040 0 -0.1453" />
+        </collision>
+    </link>
+    <joint name="axis_d" type="revolute">
+        <parent link="m2_1_1_link"/>
+        <child link="m2_joint_link"/>
+        <origin xyz="-0.02 0 0.033" rpy="0 1.56 0"/>
+        <axis xyz="0 1 0"/>
+        <limit effort="20" lower="0.0" upper="1.56" velocity="4.0"/>
+        <dynamics damping="0.1"/>
+    </joint>
+    <link name="m2_1_2_link">
+        <inertial>
+            <mass value="0.5" />
+            <inertia  ixx="0.001" ixy="0.0"  ixz="0.0"  iyy="0.001"  iyz="0.0"  izz="0.0001" />
+        </inertial>
+        <visual>
+            <geometry>
+                <mesh filename="package://bpl_alpha_description/meshes/M2-1-3.stl"/>
+            </geometry>
+            <origin rpy="0 0 0" xyz="0 0 0"/>
+            <material name="black"/>
+        </visual>
+        <collision>
+            <geometry>
+                <cylinder length="0.033" radius="0.020" />
+            </geometry>
+            <origin rpy="0 0 0" xyz="0.02 0 0.0165" />
+        </collision>
+    </link>
+    <joint name="axis_c" type="revolute">
+        <parent link="m2_joint_link"/>
+        <child link="m2_1_2_link"/>
+        <origin xyz="-0.04 0 -0.1453" rpy="0 0 3.14159"/>
+        <axis xyz="0 1 0"/>
+        <limit effort="10" lower="0.0" upper="3.5" velocity="4.0"/>
+        <dynamics damping="0.1"/>
+    </joint>
+    <link name="m1_link">
+        <inertial>
+            <mass value="0.5" />
+            <inertia  ixx="0.001" ixy="0.0"  ixz="0.0"  iyy="0.001"  iyz="0.0"  izz="0.0001" />
+        </inertial>
+        <visual>
+            <geometry>
+                <mesh filename="package://bpl_alpha_description/meshes/RS1-100-101-123.stl"/>
+            </geometry>
+            <origin rpy="0 -1.5707 0" xyz="0 0 0"/>
+            <material name="black"/>
+        </visual>
+            <collision>
+            <geometry>
+                <cylinder length="0.10975" radius="0.020" />
+            </geometry>
+            <origin rpy="0 0 0" xyz="0.00 0 0.054875" />
+        </collision>
+    </link>
+    <joint name="axis_b" type="revolute">
+        <parent link="m2_1_2_link"/>
+        <child link="m1_link"/>
+        <origin xyz="0.02 0 0.033" rpy="0 0 2.09439"/>
+        <axis xyz="0 0 -1"/>
+        <limit effort="10" lower="0.0" upper="6.2" velocity="4.0"/>
+        <dynamics damping="0.1"/>
+    </joint>
+    <joint name="jaws_joint" type="fixed">
+        <origin rpy="0 0 0" xyz="0 0 0.09975"/>
+        <parent link="m1_link"/>
+        <child link="jaws_base_link"/>
+    </joint>
+    <link name="jaws_base_link">
+        <inertial>
+            <mass value="0.5" />
+            <inertia  ixx="0.001" ixy="0.0"  ixz="0.0"  iyy="0.001"  iyz="0.0"  izz="0.0001" />
+        </inertial>
+    </link>
+    <link name="push_rod">
+        <inertial>
+            <mass value="0.2" />
+            <inertia  ixx="0.001" ixy="0.0"  ixz="0.0"  iyy="0.001"  iyz="0.0"  izz="0.0001" />
+        </inertial>
+    </link>
+    <joint name="axis_a" type="prismatic">
+        <origin rpy="0 0 0" xyz="0 0 0.009"/>
+        <parent link="jaws_base_link"/>
+        <child link="push_rod"/>
+        <axis xyz="0 0 1"/>
+        <limit effort="10" lower="0.0" upper="0.015" velocity="4.0"/>
+        <dynamics damping="0.1"/>
+    </joint>
+    <xacro:include filename="$(find bpl_alpha_description)/urdf/end_effectors/standard_jaws.urdf.xacro"/>
+    <xacro:alpha_standard_jaws parent="jaws_base_link" name="standard_jaws" axis_a="axis_a">
+        <origin xyz="0 0 0" rpy="0 0 0"/>
+    </xacro:alpha_standard_jaws>
+    <!--Included macro for end-effector-->
+    <!-- <joint name="standard_jaws_joint" type="fixed">
+        <parent link="jaws_base_link"/>
+        <child link="standard_jaws_base_link" />
+        <origin xyz="0 0 0" rpy="0 0 0"/>
+    </joint>
+    <link name="standard_jaws_base_link">
+        <visual>
+            <geometry>
+                <mesh filename="package://bpl_alpha_description/meshes/end_effectors/RS1-124.stl"/>
+            </geometry>
+            <material name="black"/>
+        </visual>
+        <inertial>
+            <mass value="0.2" />
+            <inertia  ixx="0.001" ixy="0.0"  ixz="0.0"  iyy="0.001"  iyz="0.0"  izz="0.0001" />
+        </inertial>
+    </link>
+    <link name="rs1_130_link">
+        <visual>
+            <geometry>
+                <mesh filename="package://bpl_alpha_description/meshes/end_effectors/RS1-130.stl"/>
+            </geometry>
+            <material name="black"/>
             <origin xyz="0 0 0" rpy="0 0 0"/>
-        </joint>
-        <material name="alpha_black">
-            <color rgba="0.3 0.3 0.3 1"/>
-        </material>
-        <link name="${name}_base_link"/>
-        <link name="${name}_m3_inline_link">
-            <visual>
-                <geometry>
-                    <mesh filename="package://bpl_alpha_description/meshes/M3-INLINE.stl"/>
-                </geometry>
-                <origin rpy="0 0 0" xyz="0 0 0"/>
-                <material name="alpha_black"/>
-            </visual>
-            <collision>
-                <geometry>
-                    <cylinder length="0.150" radius="0.020" />
-                </geometry>
-                <origin rpy="0 1.57075 0" xyz="-0.075 0 0" />
-            </collision>
-        </link>
-        <joint name="${name}_base_link_joint" type="fixed">
-            <parent link="${name}_base_link"/>
-            <child link="${name}_m3_inline_link"/>
-            <origin rpy="0 0 0"/>
-        </joint>
-        <link name="${name}_m2_1_1_link">
-            <visual>
-                <geometry>
-                    <mesh filename="package://bpl_alpha_description/meshes/M2-1-1.stl"/>
-                </geometry>
-                <origin rpy="0 0 0" xyz="0 0 0"/>
-                <material name="${name}_black"/>
-            </visual>
-            <collision>
-                <geometry>
-                    <cylinder length="0.066" radius="0.020" />
-                </geometry>
-                <origin rpy="0 0 0" xyz="0 0 0.000" />
-            </collision>
-        </link>
-        <joint name="${name}_axis_e" type="revolute">
-            <parent link="${name}_m3_inline_link"/>
-            <child link="${name}_m2_1_1_link"/>
-            <origin xyz="0 0 0.014"/>
-            <axis xyz="0 0 1"/>
-            <limit effort="9.0" lower="0.0" upper="6.3" velocity="0.5"/>
-        </joint>
-        <link name="${name}_m2_joint_link">
-            <visual>
-                <geometry>
-                    <mesh filename="package://bpl_alpha_description/meshes/M2.stl"/>
-                </geometry>
-                <origin rpy="0 0 0" xyz="0 0 0"/>
-                <material name="${name}_black"/>
-            </visual>
-            <collision>
-                <geometry>
-                    <cylinder length="0.145" radius="0.020" />
-                </geometry>
-                <origin rpy="0 0 0" xyz="-0.02 0 -0.0725" />
-            </collision>
-            <collision>
-                <geometry>
-                    <cylinder length="0.040" radius="0.020" />
-                </geometry>
-                <origin rpy="1.5707 0 0" xyz="0 0 0" />
-            </collision>
-            <collision>
-                <geometry>
-                    <cylinder length="0.040" radius="0.020" />
-                </geometry>
-                <origin rpy="1.5707 0 0" xyz="-0.040 0 -0.1453" />
-            </collision>
-        </link>
-        <joint name="${name}_axis_d" type="revolute">
-            <parent link="${name}_m2_1_1_link"/>
-            <child link="${name}_m2_joint_link"/>
-            <origin xyz="-0.02 0 0.033"/>
-            <axis xyz="0 1 0"/>
-            <limit effort="9.0" lower="0.0" upper="3.8" velocity="0.5"/>
-        </joint>
-        <link name="${name}_m2_1_2_link">
-            <visual>
-                <geometry>
-                    <mesh filename="package://bpl_alpha_description/meshes/M2-1-3.stl"/>
-                </geometry>
-                <origin rpy="0 0 0" xyz="0 0 0"/>
-                <material name="${name}_black"/>
-            </visual>
-            <collision>
-                <geometry>
-                    <cylinder length="0.033" radius="0.020" />
-                </geometry>
-                <origin rpy="0 0 0" xyz="0.02 0 0.0165" />
-            </collision>
-        </link>
-        <joint name="${name}_axis_c" type="revolute">
-            <parent link="${name}_m2_joint_link"/>
-            <child link="${name}_m2_1_2_link"/>
-            <origin xyz="-0.04 0 -0.1453" rpy="0 0 3.14159"/>
-            <axis xyz="0 1 0"/>
-            <limit effort="9.0" lower="0.0" upper="3.5" velocity="0.5"/>
-        </joint>
-        <link name="${name}_m1_link">
-            <visual>
-                <geometry>
-                    <mesh filename="package://bpl_alpha_description/meshes/RS1-100-101-123.stl"/>
-                </geometry>
-                <origin rpy="0 -1.5707 0" xyz="0 0 0"/>
-                <material name="${name}_black"/>
-            </visual>
-            <collision>
-                <geometry>
-                    <cylinder length="0.10975" radius="0.020" />
-                </geometry>
-                <origin rpy="0 0 0" xyz="0.00 0 0.054875" />
-            </collision>
-        </link>
-            <joint name="${name}_axis_b" type="revolute">
-            <parent link="${name}_m2_1_2_link"/>
-            <child link="${name}_m1_link"/>
-            <origin xyz="0.02 0 0.033" rpy="0 0 2.09439"/>
-            <axis xyz="0 0 -1"/>
-            <limit effort="9.0" lower="0.0" upper="6.2" velocity="0.5"/>
-        </joint>
-        <material name="${name}_jaws_black">
-            <color rgba="0.3 0.3 0.3 1"/>
-        </material>
-        <joint name="${name}_jaws_joint" type="fixed">
-            <origin rpy="0 0 0" xyz="0 0 0.09975"/>
-            <parent link="${name}_m1_link"/>
-            <child link="${name}_jaws_base_link"/>
-        </joint>
-        <link name="${name}_jaws_base_link">
-        </link>
-        <link name="${name}_push_rod"/>
-        <joint name="${name}_axis_a" type="prismatic">
-            <origin rpy="0 0 0" xyz="0 0 0.009"/>
-            <parent link="${name}_jaws_base_link"/>
-            <child link="${name}_push_rod"/>
-            <axis xyz="0 0 1"/>
-            <limit effort="10" lower="0" upper="0.015" velocity="10"/>
-        </joint>
-        <xacro:include filename="$(find bpl_alpha_description)/urdf/end_effectors/standard_jaws.urdf.xacro"/>
-        <xacro:alpha_standard_jaws parent="${name}_jaws_base_link" name="${name}_standard_jaws" axis_a="${name}_axis_a">
+        </visual>
+        <collision>
+            <origin xyz="0 0 0.01501" rpy="-0.2 0 0"/>
+            <geometry>
+                <box size="0.01 0.01 0.03"/>
+            </geometry>
+        </collision>
+        <collision>
+            <origin xyz="0 0 0.04504" rpy="0 0 0"/>
+            <geometry>
+                <box size="0.01 0.01 0.03"/>
+            </geometry>
+        </collision>
+        <collision>
+            <origin xyz="0 -0.01 0.07506" rpy="0.4  0 0"/>
+            <geometry>
+                <box size="0.01 0.01 0.03"/>
+            </geometry>
+        </collision>
+        <inertial>
+            <origin xyz="0 0 0.04505" rpy="0 0 0"/>
+            <mass value="0.1"/>
+            <inertia
+            ixx="1e-4" ixy="0.0" ixz="0.0"
+            iyy="1e-4" iyz="0.0"
+            izz="1e-4"/>
+        </inertial>
+    </link>
+    <joint name="rs1_130_joint" type="revolute">
+        <origin xyz="0 0.0155 0.0069" rpy="0 0 0"/>
+        <parent link="standard_jaws_base_link"/>
+        <child link="rs1_130_link"/>
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
File: ROS2/bpl_alpha_description/urdf/end_effectors/standard_jaws.urdf.xacro (robot description, xacro)
@@ -18,4 +18,8 @@
                 <material name="${name}_black"/>
             </visual>
+            <inertial>
+                <mass value="0.2" />
+                <inertia  ixx="0.001" ixy="0.0"  ixz="0.0"  iyy="0.001"  iyz="0.0"  izz="0.0001" />
+            </inertial>
         </link>
         <link name="${name}_rs1_130_link">
@@ -24,13 +28,33 @@
                     <mesh filename="package://bpl_alpha_description/meshes/end_effectors/RS1-130.stl"/>
                 </geometry>
-                <material name="${name}_black"/>
-                <origin xyz="0 0 0" rpy="0 0 0"/>
-            </visual>
-            <collision>
-                <geometry>
-                    <box size="0.012 0.03 0.09"/>
-                </geometry>
-                <origin xyz="0.0 -0.008 0.045" rpy="0 0 0"/>
-            </collision>
+            <material name="${name}_black"/>
+            <origin xyz="0 0 0" rpy="0 0 0"/>
+        </visual>
+        <collision>
+            <origin xyz="0 0 0.01501" rpy="-0.2 0 0"/>
+            <geometry>
+                <box size="0.01 0.01 0.03"/>
+            </geometry>
+        </collision>
+        <collision>
+            <origin xyz="0 0 0.04504" rpy="0 0 0"/>
+            <geometry>
+                <box size="0.01 0.01 0.03"/>
+            </geometry>
+        </collision>
+        <collision>
+            <origin xyz="0 -0.01 0.07506" rpy="0.4  0 0"/>
+            <geometry>
+                <box size="0.01 0.01 0.03"/>
+            </geometry>
+        </collision>
+        <inertial>
+            <origin xyz="0 0 0.04505" rpy="0 0 0"/>
+            <mass value="0.1"/>
+            <inertia
+            ixx="1e-4" ixy="0.0" ixz="0.0"
+            iyy="1e-4" iyz="0.0"
+            izz="1e-4"/>
+        </inertial>
         </link>
         <joint name="${name}_rs1_130_joint" type="revolute">
@@ -47,13 +71,33 @@
                     <mesh filename="package://bpl_alpha_description/meshes/end_effectors/RS1-139.stl"/>
                 </geometry>
-                <material name="${name}_black"/>
-                <origin xyz="0 0 0" rpy="0 0 0"/>
-            </visual>
-            <collision>
-                <geometry>
-                    <box size="0.012 0.03 0.09"/>
-                </geometry>
-                <origin xyz="0.0 0.008 0.045" rpy="0 0 0"/>
-            </collision>
+            <material name="${name}_black"/>
+            <origin xyz="0 0 0" rpy="0 0 0"/>
+        </visual>
+        <collision>
+            <origin xyz="0 0 0.01501" rpy="0.2 0 0"/>
+            <geometry>
+                <box size="0.01 0.01 0.03"/>
+            </geometry>
+        </collision>
+        <collision>
+            <origin xyz="0 0 0.04504" rpy="0 0 0"/>
+            <geometry>
+                <box size="0.01 0.01 0.03"/>
+            </geometry>
+        </collision>
+        <collision>
+            <origin xyz="0 0.01 0.07506" rpy="-0.4  0 0"/>
+            <geometry>
+                <box size="0.01 0.01 0.03"/>
+            </geometry>
+        </collision>
+        <inertial>
+            <origin xyz="0 0 0.04505" rpy="0 0 0"/>
+            <mass value="0.1"/>
+            <inertia
+            ixx="1e-4" ixy="0.0" ixz="0.0"
+            iyy="1e-4" iyz="0.0"
+            izz="1e-4"/>
+        </inertial>
         </link>
         <joint name="${name}_rs1_139_joint" type="revolute">
@@ -65,4 +109,13 @@
           <mimic joint="${name}_rs1_130_joint" multiplier="1" offset="0"/>
         </joint>
+        <gazebo reference="${name}_base_link">
+            <material>Gazebo/FlatBlack</material>
+        </gazebo>
+        <gazebo reference="${name}_rs1_130_link">
+            <material>Gazebo/FlatBlack</material>
+        </gazebo>
+        <gazebo reference="${name}_rs1_139_link">
+            <material>Gazebo/FlatBlack</material>
+        </gazebo>
     </xacro:macro>
 </robot>

File: ROS2/bpl_alpha_description/urdf/ros2_control.xacro (robot description, xacro)
@@ -1,17 +1,4 @@
 <?xml version="1.0"?>
 <robot xmlns:xacro="http://ros.org/wiki/xacro">
-  <!-- Macro to create a SimpleTransmission block -->
-  <xacro:macro name="add_transmission" params="joint_name">
-    <transmission name="${joint_name}_trans">
-      <type>transmission_interface/SimpleTransmission</type>
-      <joint name="${joint_name}">
-        <hardwareInterface>hardware_interface/PositionJointInterface</hardwareInterface>
-      </joint>
-      <actuator name="${joint_name}_motor">
-        <hardwareInterface>hardware_interface/PositionJointInterface</hardwareInterface>
-        <mechanicalReduction>1</mechanicalReduction>
-      </actuator>
-    </transmission>
-  </xacro:macro>
   <!-- ros2_control hardware interface block -->
   <ros2_control name="GazeboSystem" type="system">
@@ -19,25 +6,25 @@
       <plugin>gz_ros2_control/GazeboSimSystem</plugin>
     </hardware>
-    <joint name="alpha_axis_a">
+    <joint name="axis_a">
       <command_interface name="position"/>
       <state_interface name="position"/>
       <state_interface name="velocity"/>
     </joint>
-    <joint name="alpha_axis_b">
+    <joint name="axis_b">
       <command_interface name="position"/>
       <state_interface name="position"/>
       <state_interface name="velocity"/>
     </joint>
-    <joint name="alpha_axis_c">
+    <joint name="axis_c">
       <command_interface name="position"/>
       <state_interface name="position"/>
       <state_interface name="velocity"/>
     </joint>
-    <joint name="alpha_axis_d">
+    <joint name="axis_d">
       <command_interface name="position"/>
       <state_interface name="position"/>
       <state_interface name="velocity"/>
     </joint>
-    <joint name="alpha_axis_e">
+    <joint name="axis_e">
       <command_interface name="position"/>
       <state_interface name="position"/>
