Commit message: Fix joint values in alpha_5.urdf.xacro

File: ROS2/bpl_alpha_description/urdf/alpha_5.urdf.xacro (robot description, xacro)
@@ -66,5 +66,5 @@
         <origin xyz="0 0 0.014"/>
         <axis xyz="0 0 1"/>
-        <limit effort="25" lower="0.0" upper="6.3" velocity="4.0"/>
+        <limit effort="25" lower="0.0" upper="6.3" velocity="0.5"/>
         <dynamics damping="0.1"/>
     </joint>
@@ -103,7 +103,7 @@
         <parent link="m2_1_1_link"/>
         <child link="m2_joint_link"/>
-        <origin xyz="-0.02 0 0.033" rpy="0 1.56 0"/>
+        <origin xyz="-0.02 0 0.033"/>
         <axis xyz="0 1 0"/>
-        <limit effort="20" lower="0.0" upper="1.56" velocity="4.0"/>
+        <limit effort="20" lower="0.0" upper="3.8" velocity="0.5"/>
         <dynamics damping="0.1"/>
     </joint>
@@ -132,5 +132,5 @@
         <origin xyz="-0.04 0 -0.1453" rpy="0 0 3.14159"/>
         <axis xyz="0 1 0"/>
-        <limit effort="10" lower="0.0" upper="3.5" velocity="4.0"/>
+        <limit effort="10" lower="0.0" upper="3.5" velocity="0.5"/>
         <dynamics damping="0.1"/>
     </joint>
@@ -159,5 +159,5 @@
         <origin xyz="0.02 0 0.033" rpy="0 0 2.09439"/>
         <axis xyz="0 0 -1"/>
-        <limit effort="10" lower="0.0" upper="6.2" velocity="4.0"/>
+        <limit effort="10" lower="0.0" upper="6.2" velocity="0.5"/>
         <dynamics damping="0.1"/>
     </joint>
@@ -184,5 +184,5 @@
         <child link="push_rod"/>
         <axis xyz="0 0 1"/>
-        <limit effort="10" lower="0.0" upper="0.015" velocity="4.0"/>
+        <limit effort="10" lower="0.0" upper="0.015" velocity="10.0"/>
         <dynamics damping="0.1"/>
     </joint>

Commit message: minor fixes in bpl_alpha_description package

File: ROS2/bpl_alpha_description/urdf/alpha_5.urdf.xacro (robot description, xacro)
@@ -191,117 +191,4 @@
         <origin xyz="0 0 0" rpy="0 0 0"/>
     </xacro:alpha_standard_jaws>
-    <!--Included macro for end-effector-->
-    <!-- <joint name="standard_jaws_joint" type="fixed">
-        <parent link="jaws_base_link"/>
-        <child link="standard_jaws_base_link" />
-        <origin xyz="0 0 0" rpy="0 0 0"/>
-    </joint>
-    <link name="standard_jaws_base_link">
-        <visual>
-            <geometry>
-                <mesh filename="package://bpl_alpha_description/meshes/end_effectors/RS1-124.stl"/>
-            </geometry>
-            <material name="black"/>
-        </visual>
-        <inertial>
-            <mass value="0.2" />
-            <inertia  ixx="0.001" ixy="0.0"  ixz="0.0"  iyy="0.001"  iyz="0.0"  izz="0.0001" />
-        </inertial>
-    </link>
-    <link name="rs1_130_link">
-        <visual>
-            <geometry>
-                <mesh filename="package://bpl_alpha_description/meshes/end_effectors/RS1-130.stl"/>
-            </geometry>
-            <material name="black"/>
-            <origin xyz="0 0 0" rpy="0 0 0"/>
-        </visual>
-        <collision>
-            <origin xyz="0 0 0.01501" rpy="-0.2 0 0"/>
-            <geometry>
-                <box size="0.01 0.01 0.03"/>
-            </geometry>
-        </collision>
-        <collision>
-            <origin xyz="0 0 0.04504" rpy="0 0 0"/>
-            <geometry>
-                <box size="0.01 0.01 0.03"/>
-            </geometry>
-        </collision>
-        <collision>
-            <origin xyz="0 -0.01 0.07506" rpy="0.4  0 0"/>
-            <geometry>
-                <box size="0.01 0.01 0.03"/>
-            </geometry>
-        </collision>
-        <inertial>
-            <origin xyz="0 0 0.04505" rpy="0 0 0"/>
-            <mass value="0.1"/>
-            <inertia
-            ixx="1e-4" ixy="0.0" ixz="0.0"
-            iyy="1e-4" iyz="0.0"
-            izz="1e-4"/>
-        </inertial>
-    </link>
-    <joint name="rs1_130_joint" type="revolute">
-        <origin xyz="0 0.0155 0.0069" rpy="0 0 0"/>
-        <parent link="standard_jaws_base_link"/>
-        <child link="rs1_130_link"/>
-        <axis xyz="-1 0 0"/>
-        <limit lower="0" upper="0.5" effort="10" velocity="10"/>
-        <mimic joint="axis_a" multiplier="51" offset="0"/>
-    </joint>
-    <link name="rs1_139_link">
-        <visual>
-            <geometry>
-                <mesh filename="package://bpl_alpha_description/meshes/end_effectors/RS1-139.stl"/>
-            </geometry>
-            <material name="black"/>
-            <origin xyz="0 0 0" rpy="0 0 0"/>
-        </visual>
-        <collision>
-            <origin xyz="0 0 0.01501" rpy="0.2 0 0"/>
-            <geometry>
-                <box size="0.01 0.01 0.03"/>
-            </geometry>
-        </collision>
-        <collision>
-            <origin xyz="0 0 0.04504" rpy="0 0 0"/>
-            <geometry>
-                <box size="0.01 0.01 0.03"/>
-            </geometry>
-        </collision>
-        <collision>
-            <origin xyz="0 0.01 0.07506" rpy="-0.4  0 0"/>
-            <geometry>
-                <box size="0.01 0.01 0.03"/>
-            </geometry>
-        </collision>
-        <inertial>
-            <origin xyz="0 0 0.04505" rpy="0 0 0"/>
-            <mass value="0.1"/>
-            <inertia
-            ixx="1e-4" ixy="0.0" ixz="0.0"
-            iyy="1e-4" iyz="0.0"
-            izz="1e-4"/>
-        </inertial>
-    </link>
-    <joint name="rs1_139_joint" type="revolute">
-        <origin xyz="0 -0.0155 0.0069" rpy="0 0 0"/>
-        <parent link="standard_jaws_base_link"/>
-        <child link="rs1_139_link"/>
-        <axis xyz="1 0 0"/>
-        <limit lower="0" upper="0.5" effort="10" velocity="10"/>
-        <mimic joint="rs1_130_joint" multiplier="1" offset="0"/>
-    </joint> -->
-    <!-- <gazebo reference="standard_jaws_base_link">
-        <material>Gazebo/FlatBlack</material>
-    </gazebo>
-    <gazebo reference="rs1_130_link">
-        <material>Gazebo/FlatBlack</material>
-    </gazebo>
-    <gazebo reference="rs1_139_link">
-        <material>Gazebo/FlatBlack</material>
-    </gazebo> -->
     <gazebo reference="m3_inline_link">
         <material>Gazebo/FlatBlack</material>
@@ -319,4 +206,5 @@
         <material>Gazebo/FlatBlack</material>
     </gazebo>
+    <xacro:arg name="sim_mode" default="true"/>
     <xacro:include filename='ros2_control.xacro'/>
 </robot>

File: ROS2/bpl_alpha_description/urdf/ros2_control.xacro (robot description, xacro)
@@ -1,35 +1,69 @@
 <?xml version="1.0"?>
 <robot xmlns:xacro="http://ros.org/wiki/xacro">
-  <!-- ros2_control hardware interface block -->
-  <ros2_control name="GazeboSystem" type="system">
-    <hardware>
-      <plugin>gz_ros2_control/GazeboSimSystem</plugin>
-    </hardware>
-    <joint name="axis_a">
-      <command_interface name="position"/>
-      <state_interface name="position"/>
-      <state_interface name="velocity"/>
-    </joint>
-    <joint name="axis_b">
-      <command_interface name="position"/>
-      <state_interface name="position"/>
-      <state_interface name="velocity"/>
-    </joint>
-    <joint name="axis_c">
-      <command_interface name="position"/>
-      <state_interface name="position"/>
-      <state_interface name="velocity"/>
-    </joint>
-    <joint name="axis_d">
-      <command_interface name="position"/>
-      <state_interface name="position"/>
-      <state_interface name="velocity"/>
-    </joint>
-    <joint name="axis_e">
-      <command_interface name="position"/>
-      <state_interface name="position"/>
-      <state_interface name="velocity"/>
-    </joint>
-  </ros2_control>
+  <xacro:if value="$(arg sim_mode)">
+    <ros2_control name="GazeboSystem" type="system">
+      <hardware>
+        <plugin>gz_ros2_control/GazeboSimSystem</plugin>
+      </hardware>
+      <joint name="axis_a">
+        <command_interface name="position"/>
+        <state_interface name="position"/>
+        <state_interface name="velocity"/>
+      </joint>
+      <joint name="axis_b">
+        <command_interface name="position"/>
+        <state_interface name="position"/>
+        <state_interface name="velocity"/>
+      </joint>
+      <joint name="axis_c">
+        <command_interface name="position"/>
+        <state_interface name="position"/>
+        <state_interface name="velocity"/>
+      </joint>
+      <joint name="axis_d">
+        <command_interface name="position"/>
+        <state_interface name="position"/>
+        <state_interface name="velocity"/>
+      </joint>
+      <joint name="axis_e">
+        <command_interface name="position"/>
+        <state_interface name="position"/>
+        <state_interface name="velocity"/>
+      </joint>
+    </ros2_control>
+  </xacro:if>
+  <xacro:unless value="$(arg sim_mode)">
+    <ros2_control name="RealRobot" type="system">
+      <hardware>
+        <plugin>alpha_5_hardware/Alpha5HardwareInterface</plugin>
+        <param name="manipulator_serial_port">/dev/ttyUSB0</param>
+      </hardware>
+      <joint name="axis_a">
+        <command_interface name="position"/>
+        <state_interface name="position"/>
+        <state_interface name="velocity"/>
+      </joint>
+      <joint name="axis_b">
+        <command_interface name="position"/>
+        <state_interface name="position"/>
+        <state_interface name="velocity"/>
+      </joint>
+      <joint name="axis_c">
+        <command_interface name="position"/>
+        <state_interface name="position"/>
+        <state_interface name="velocity"/>
+      </joint>
+      <joint name="axis_d">
+        <command_interface name="position"/>
+        <state_interface name="position"/>
+        <state_interface name="velocity"/>
+      </joint>
+      <joint name="axis_e">
+        <command_interface name="position"/>
+        <state_interface name="position"/>
+        <state_interface name="velocity"/>
+      </joint>
+    </ros2_control>
+  </xacro:unless>
   <gazebo>
     <plugin name="gz_ros2_control::GazeboSimROS2ControlPlugin" filename="libgz_ros2_control-system.so">
